File: boards/balancing_robot_h_bridges_power_sup.brd (EAGLE design)
At the start: 35 x 75 mm, 16 parts

Commit message: finished h-bridges and psu board, rev. 1
Parts:
- removed JP4: (no value), pinhead:1X20
- added C3, C7: 10u, rcl:153CLV-0405
- added C6: 100n, rcl:C0603
- added JP1: (no value), pinhead:1X24
- moved C4 32.3 mm to (18.0, 50.5), turned to 0 degrees
- moved C1 27.6 mm to (26.2, 55.4)
- moved C8 27.3 mm to (27.5, 50.5), turned to 180 degrees
- moved C5 14.6 mm to (19.3, 44.6)
- moved C2 12.0 mm to (26.3, 44.6)
- moved R1 2.24 mm to (32.0, 5.00), turned to 0 degrees
- moved LED1 1.12 mm to (32.0, 3.00), turned to 270 degrees
Connections:
- removed net N$11: JP4.6
- removed net N$12: JP4.7
- removed net N$13: JP4.8
- removed net N$14: JP4.9
- removed net N$15: JP4.10
- removed net N$6: JP4.3
- removed net N$7: JP4.4
- net ENK_MOTOR1A: now also JP1.18; no longer JP4.14
- net ENK_MOTOR1B: now also JP1.17; no longer JP4.13
- net ENK_MOTOR2A: now also JP1.16; no longer JP4.12
- net ENK_MOTOR2B: now also JP1.15; no longer JP4.11
- net GND: now also C3.-, C6.1, C7.-, JP1.5, JP1.6; no longer JP4.5
- net MOTOR1_1: now also JP1.19; no longer JP4.19
- net MOTOR1_2: now also JP1.20; no longer JP4.18
- net MOTOR1_PWM: now also JP1.21; no longer JP4.20
- net MOTOR2_1: now also JP1.22; no longer JP4.16
- net MOTOR2_2: now also JP1.23; no longer JP4.15
- net MOTOR2_PWM: now also JP1.24; no longer JP4.17
- net VCC: now also C3.+, C6.2, C7.+, JP1.1, JP1.2, JP1.3, JP1.4; no longer JP4.1, JP4.2
Routing:
- net VCC: track 170.9 -> 228.4 mm, vias 3 -> 6
- net ENK_MOTOR2A: track 0.00 -> 25.3 mm
- net GND: track 23.4 -> 0.00 mm, vias 2 -> 0
- net MOTOR1_PWM: track 10.5 -> 32.9 mm
- net ENK_MOTOR2B: track 0.00 -> 21.8 mm
- net ENK_MOTOR1B: track 0.00 -> 21.4 mm
- net MOTOR2_PWM: track 10.5 -> 31.7 mm
- net ENK_MOTOR1A: track 0.00 -> 20.7 mm
- net MOTOR1_2: track 8.37 -> 29.0 mm
- net MOTOR2_2: track 8.42 -> 27.8 mm
- net MOTOR1_1: track 6.24 -> 25.1 mm
- net MOTOR2_1: track 6.29 -> 23.9 mm
- added copper zone on layer 16, net N$1
- added copper zone on layer 1, net N$2

Commit message: updated bridge board
Parts:
- moved C8 0.63 mm to (28.1, 50.5)
- moved C6 0.52 mm to (19.1, 55.2), turned to 180 degrees
- moved C3 0.22 mm to (17.8, 61.0)
Connections:
- removed net N$5: U$3.10, U$3.3, U$3.4, U$3.9, U$6.10, U$6.3, U$6.4, U$6.9
- net GND: now also C6.2, U$3.10, U$3.3, U$3.4, U$3.9, U$6.10, U$6.3, U$6.4, U$6.9; no longer C6.1
- net VCC: now also C6.1; no longer C6.2
Routing:
- net VCC: track 228.4 -> 253.0 mm, vias 6 -> 7
- net ENK_MOTOR1A: track 20.7 -> 24.9 mm
- net OUT_MOTOR2_1: track 54.1 -> 57.5 mm, vias 2 -> 4
- net OUT_MOTOR1_1: track 26.1 -> 29.5 mm, vias 2 -> 4
- net OUT_MOTOR1_2: track 15.0 -> 16.8 mm, vias 1 -> 2
- net OUT_MOTOR2_2: track 37.8 -> 39.4 mm, vias 1 -> 2
- added copper zone on layer 1, net GND
- added copper zone on layer 16, net GND
- removed copper zone on layer 16, net N$1
- removed copper zone on layer 1, net N$2
