File: boards/balancing_robot_psoc.sch (EAGLE design)
At the start: 28 parts

Commit message: added capacitors on power sup line on psoc board
Parts:
- added C1: (no value), rcl:C-EUC0603
- added C2: (no value), rcl:C-EUC0805
Connections:
- net GND: now also C1.2, C2.2
- net POWER_SUP: now also C1.1, C2.1
Changed lines of the file:
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@@
 <part name="R16" library="rcl" deviceset="R-EU_" device="R0603"/>
 <part name="R17" library="rcl" deviceset="R-EU_" device="R0603"/>
+<part name="C1" library="rcl" deviceset="C-EU" device="C0603"/>
+<part name="C2" library="rcl" deviceset="C-EU" device="C0805"/>
+<part name="GND6" library="supply1" deviceset="GND" device=""/>
 </parts>
 <sheets>
@@
 <instance part="R16" gate="G$1" x="177.8" y="127" rot="R90"/>
 <instance part="R17" gate="G$1" x="139.7" y="142.24" rot="R180"/>
+<instance part="C1" gate="G$1" x="195.58" y="124.46"/>
+<instance part="C2" gate="G$1" x="205.74" y="124.46"/>
+<instance part="GND6" gate="1" x="200.66" y="111.76"/>
 </instances>
 <busses>
@@
 <wire x1="33.02" y1="76.2" x2="33.02" y2="71.12" width="0.1524" layer="91"/>
 </segment>
+<segment>
+<pinref part="C2" gate="G$1" pin="2"/>
+<wire x1="205.74" y1="119.38" x2="205.74" y2="116.84" width="0.1524" layer="91"/>
+<wire x1="205.74" y1="116.84" x2="200.66" y2="116.84" width="0.1524" layer="91"/>
+<pinref part="C1" gate="G$1" pin="2"/>
+<wire x1="200.66" y1="116.84" x2="195.58" y2="116.84" width="0.1524" layer="91"/>
+<wire x1="195.58" y1="116.84" x2="195.58" y2="119.38" width="0.1524" layer="91"/>
+<wire x1="200.66" y1="116.84" x2="200.66" y2="114.3" width="0.1524" layer="91"/>
+<junction x="200.66" y="116.84"/>
+<pinref part="GND6" gate="1" pin="GND"/>
+</segment>
 </net>
 <net name="VCC" class="0">
@@
 <wire x1="134.62" y1="142.24" x2="132.08" y2="142.24" width="0.1524" layer="91"/>
 <label x="132.08" y="142.24" size="1.27" layer="95" rot="R180" xref="yes"/>
-</segment>
-</net>
+<label x="200.66" y="132.08" size="1.27" layer="95" rot="R180" xref="yes"/>
+</segment>
+<segment>
+<pinref part="C1" gate="G$1" pin="1"/>
+<wire x1="195.58" y1="127" x2="195.58" y2="129.54" width="0.1524" layer="91"/>
+<wire x1="195.58" y1="129.54" x2="200.66" y2="129.54" width="0.1524" layer="91"/>
+<pinref part="C2" gate="G$1" pin="1"/>
+<wire x1="200.66" y1="129.54" x2="205.74" y2="129.54" width="0.1524" layer="91"/>
+<wire x1="205.74" y1="129.54" x2="205.74" y2="127" width="0.1524" layer="91"/>
+<wire x1="200.66" y1="129.54" x2="200.66" y2="132.08" width="0.1524" layer="91"/>
+<junction x="200.66" y="129.54"/>
+</segment>
+</net>

Commit message: final changes of boards - production version
Parts:
- added C3: (no value), rcl:C-EUC0603
Connections:
- net GND: now also C3.2
- net N$2: now also C3.1
Other:
- moved on the sheet: R5
Changed lines of the file:
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@@
 <part name="C2" library="rcl" deviceset="C-EU" device="C0805"/>
 <part name="GND6" library="supply1" deviceset="GND" device=""/>
+<part name="C3" library="rcl" deviceset="C-EU" device="C0603"/>
+<part name="GND7" library="supply1" deviceset="GND" device=""/>
 </parts>
 <sheets>
@@
 <instance part="R3" gate="G$1" x="101.6" y="43.18" rot="R180"/>
 <instance part="R4" gate="G$1" x="45.72" y="48.26" rot="R180"/>
-<instance part="R5" gate="G$1" x="45.72" y="27.94" rot="R180"/>
+<instance part="R5" gate="G$1" x="25.4" y="27.94" rot="R180"/>
 <instance part="R6" gate="G$1" x="142.24" y="5.08"/>
 <instance part="R7" gate="G$1" x="142.24" y="10.16"/>
@@
 <instance part="C2" gate="G$1" x="205.74" y="124.46"/>
 <instance part="GND6" gate="1" x="200.66" y="111.76"/>
+<instance part="C3" gate="G$1" x="40.64" y="22.86"/>
+<instance part="GND7" gate="1" x="40.64" y="12.7"/>
 </instances>
 <busses>
@@
 <pinref part="GND6" gate="1" pin="GND"/>
 </segment>
+<segment>
+<pinref part="C3" gate="G$1" pin="2"/>
+<wire x1="40.64" y1="17.78" x2="40.64" y2="15.24" width="0.1524" layer="91"/>
+<pinref part="GND7" gate="1" pin="GND"/>
+</segment>
 </net>
 <net name="VCC" class="0">
@@
 <segment>
 <pinref part="U$1" gate="G$1" pin="VREF"/>
-<wire x1="63.5" y1="27.94" x2="50.8" y2="27.94" width="0.1524" layer="91"/>
+<wire x1="63.5" y1="27.94" x2="40.64" y2="27.94" width="0.1524" layer="91"/>
 <pinref part="R5" gate="G$1" pin="1"/>
+<pinref part="C3" gate="G$1" pin="1"/>
+<wire x1="40.64" y1="27.94" x2="30.48" y2="27.94" width="0.1524" layer="91"/>
+<wire x1="40.64" y1="25.4" x2="40.64" y2="27.94" width="0.1524" layer="91"/>
+<junction x="40.64" y="27.94"/>
 </segment>
 </net>
@@
 <segment>
 <pinref part="R5" gate="G$1" pin="2"/>
-<wire x1="40.64" y1="27.94" x2="38.1" y2="27.94" width="0.1524" layer="91"/>
-<label x="38.1" y="27.94" size="1.27" layer="95" rot="R180" xref="yes"/>
-</segment>
-<segment>
+<wire x1="20.32" y1="27.94" x2="17.78" y2="27.94" width="0.1524" layer="91"/>
+<label x="17.78" y="27.94" size="1.27" layer="95" rot="R180" xref="yes"/>
+</segment>
+<segment>
