File: boards/balancing_robot_h_bridges_power_sup.sch (EAGLE design)
At the start: 16 parts

Commit message: finished h-bridges and psu board, rev. 1
Parts:
- removed JP4: (no value), pinhead:PINHD-1X20
- added C3, C7: 10u, rcl:CPOL-EU153CLV-0405
- added C6: 100n, rcl:C-EUC0603
- added JP1: (no value), pinhead:PINHD-1X24
Connections:
- removed net N$11: JP4.6
- removed net N$12: JP4.7
- removed net N$13: JP4.8
- removed net N$14: JP4.9
- removed net N$15: JP4.10
- removed net N$6: JP4.3
- removed net N$7: JP4.4
- net ENK_MOTOR1A: now also JP1.18; no longer JP4.14
- net ENK_MOTOR1B: now also JP1.17; no longer JP4.13
- net ENK_MOTOR2A: now also JP1.16; no longer JP4.12
- net ENK_MOTOR2B: now also JP1.15; no longer JP4.11
- net GND: now also C3.-, C6.1, C7.-, JP1.5, JP1.6; no longer JP4.5
- net MOTOR1_1: now also JP1.19; no longer JP4.19
- net MOTOR1_2: now also JP1.20; no longer JP4.18
- net MOTOR1_PWM: now also JP1.21; no longer JP4.20
- net MOTOR2_1: now also JP1.22; no longer JP4.16
- net MOTOR2_2: now also JP1.23; no longer JP4.15
- net MOTOR2_PWM: now also JP1.24; no longer JP4.17
- net VCC: now also C3.+, C6.2, C7.+, JP1.1, JP1.2, JP1.3, JP1.4; no longer JP4.1, JP4.2

Commit message: updated bridge board
Connections:
- removed net N$5: U$3.PGND1@3, U$3.PGND1@4, U$3.PGND2@10, U$3.PGND2@9, U$6.PGND1@3, U$6.PGND1@4, U$6.PGND2@10, U$6.PGND2@9
- net GND: now also C6.2, U$3.PGND1@3, U$3.PGND1@4, U$3.PGND2@10, U$3.PGND2@9, U$6.PGND1@3, U$6.PGND1@4, U$6.PGND2@10, U$6.PGND2@9; no longer C6.1
- net VCC: now also C6.1; no longer C6.2
Other:
- moved on the sheet: C3, C6
Changed lines of the file:
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@@
 <part name="SUPPLY1" library="supply2" deviceset="VCC" device=""/>
 <part name="VAABT" library="supply1" deviceset="VCC" device="" value="VBAT"/>
-<part name="GND4" library="supply1" deviceset="GND" device=""/>
 <part name="GND5" library="supply1" deviceset="GND" device=""/>
 <part name="SUPPLY3" library="supply2" deviceset="VCC" device=""/>
@@
 <part name="GND7" library="supply1" deviceset="GND" device=""/>
 <part name="U$6" library="SparkFun-PowerIC" deviceset="TB6612FNG" device="" value="TB6612FNG"/>
-<part name="GND8" library="supply1" deviceset="GND" device=""/>
 <part name="GND9" library="supply1" deviceset="GND" device=""/>
 <part name="SUPPLY4" library="supply2" deviceset="VCC" device=""/>
-<part name="VAABT2" library="supply1" deviceset="VCC" device="" value="VBAT"/>
+<part name="VBAT" library="supply1" deviceset="VCC" device="" value="VBAT"/>
 <part name="C5" library="rcl" deviceset="C-EU" device="C0603" value="100n"/>
 <part name="GND10" library="supply1" deviceset="GND" device=""/>
@@
 <part name="C8" library="rcl" deviceset="CPOL-EU" device="153CLV-0405" value="10u"/>
 <part name="JP1" library="pinhead" deviceset="PINHD-1X24" device=""/>
-<part name="C3" library="rcl" deviceset="CPOL-EU" device="153CLV-0405" value="10u"/>
 <part name="C7" library="rcl" deviceset="CPOL-EU" device="153CLV-0405" value="10u"/>
-<part name="C6" library="rcl" deviceset="C-EU" device="C0603" value="100n"/>
 <part name="GND3" library="supply1" deviceset="GND" device=""/>
 <part name="VAABT3" library="supply1" deviceset="VCC" device="" value="VBAT"/>
+<part name="C3" library="rcl" deviceset="CPOL-EU" device="153CLV-0405" value="10u"/>
+<part name="C6" library="rcl" deviceset="C-EU" device="C0603" value="100n"/>
+<part name="GND8" library="supply1" deviceset="GND" device=""/>
+<part name="GND4" library="supply1" deviceset="GND" device=""/>
 </parts>
 <sheets>
@@
 <instance part="SUPPLY1" gate="G$1" x="195.58" y="134.62"/>
 <instance part="VAABT" gate="VCC" x="132.08" y="137.16"/>
-<instance part="GND4" gate="1" x="25.4" y="5.08"/>
 <instance part="GND5" gate="1" x="63.5" y="5.08"/>
 <instance part="SUPPLY3" gate="G$1" x="63.5" y="66.04"/>
@@
 <instance part="GND7" gate="1" x="81.28" y="48.26"/>
 <instance part="U$6" gate="G$1" x="45.72" y="101.6"/>
-<instance part="GND8" gate="1" x="25.4" y="78.74"/>
 <instance part="GND9" gate="1" x="63.5" y="78.74"/>
 <instance part="SUPPLY4" gate="G$1" x="63.5" y="139.7"/>
-<instance part="VAABT2" gate="VCC" x="71.12" y="142.24"/>
+<instance part="VBAT" gate="VCC" x="71.12" y="142.24"/>
 <instance part="C5" gate="G$1" x="58.42" y="127" rot="R90"/>
 <instance part="GND10" gate="1" x="53.34" y="121.92"/>
@@
 <instance part="C8" gate="G$1" x="73.66" y="134.62" rot="R90"/>
 <instance part="JP1" gate="A" x="111.76" y="45.72" rot="R180"/>
-<instance part="C3" gate="G$1" x="73.66" y="127" rot="R90"/>
 <instance part="C7" gate="G$1" x="60.96" y="134.62" rot="R270"/>
-<instance part="C6" gate="G$1" x="58.42" y="60.96" rot="R90"/>
 <instance part="GND3" gate="1" x="127" y="10.16"/>
 <instance part="VAABT3" gate="VCC" x="152.4" y="27.94"/>
+<instance part="C3" gate="G$1" x="60.96" y="60.96" rot="R270"/>
+<instance part="C6" gate="G$1" x="73.66" y="127" rot="R90"/>
+<instance part="GND8" gate="1" x="25.4" y="78.74"/>
+<instance part="GND4" gate="1" x="25.4" y="5.08"/>
 </instances>
 <busses>
@@
 <junction x="53.34" y="53.34"/>
 <pinref part="GND6" gate="1" pin="GND"/>
-<pinref part="C6" gate="G$1" pin="1"/>
+<pinref part="C3" gate="G$1" pin="-"/>
 </segment>
 <segment>
@@
 <pinref part="GND11" gate="1" pin="GND"/>
 <pinref part="C8" gate="G$1" pin="-"/>
-<pinref part="C3" gate="G$1" pin="-"/>
+<pinref part="C6" gate="G$1" pin="2"/>
 </segment>
 <segment>
@@
 <junction x="124.46" y="27.94"/>
 <pinref part="GND3" gate="1" pin="GND"/>
+</segment>
+<segment>
+<pinref part="U$6" gate="G$1" pin="PGND1@3"/>
+<wire x1="27.94" y1="109.22" x2="25.4" y2="109.22" width="0.1524" layer="91"/>
+<wire x1="25.4" y1="109.22" x2="25.4" y2="106.68" width="0.1524" layer="91"/>
+<pinref part="U$6" gate="G$1" pin="PGND2@10"/>
+<wire x1="25.4" y1="106.68" x2="25.4" y2="93.98" width="0.1524" layer="91"/>
+<wire x1="25.4" y1="93.98" x2="25.4" y2="91.44" width="0.1524" layer="91"/>
+<wire x1="25.4" y1="91.44" x2="25.4" y2="81.28" width="0.1524" layer="91"/>
+<wire x1="27.94" y1="91.44" x2="25.4" y2="91.44" width="0.1524" layer="91"/>
+<junction x="25.4" y="91.44"/>
+<pinref part="U$6" gate="G$1" pin="PGND2@9"/>
+<wire x1="27.94" y1="93.98" x2="25.4" y2="93.98" width="0.1524" layer="91"/>
+<junction x="25.4" y="93.98"/>
+<pinref part="U$6" gate="G$1" pin="PGND1@4"/>
+<wire x1="27.94" y1="106.68" x2="25.4" y2="106.68" width="0.1524" layer="91"/>
+<junction x="25.4" y="106.68"/>
+<pinref part="GND8" gate="1" pin="GND"/>
+</segment>
+<segment>
+<pinref part="U$3" gate="G$1" pin="PGND1@3"/>
+<wire x1="27.94" y1="35.56" x2="25.4" y2="35.56" width="0.1524" layer="91"/>
+<wire x1="25.4" y1="35.56" x2="25.4" y2="33.02" width="0.1524" layer="91"/>
+<pinref part="U$3" gate="G$1" pin="PGND2@10"/>
+<wire x1="25.4" y1="33.02" x2="25.4" y2="20.32" width="0.1524" layer="91"/>
+<wire x1="25.4" y1="20.32" x2="25.4" y2="17.78" width="0.1524" layer="91"/>
+<wire x1="25.4" y1="17.78" x2="25.4" y2="7.62" width="0.1524" layer="91"/>
+<wire x1="27.94" y1="17.78" x2="25.4" y2="17.78" width="0.1524" layer="91"/>
+<junction x="25.4" y="17.78"/>
+<pinref part="U$3" gate="G$1" pin="PGND2@9"/>
+<wire x1="27.94" y1="20.32" x2="25.4" y2="20.32" width="0.1524" layer="91"/>
+<junction x="25.4" y="20.32"/>
+<pinref part="U$3" gate="G$1" pin="PGND1@4"/>
+<wire x1="27.94" y1="33.02" x2="25.4" y2="33.02" width="0.1524" layer="91"/>
+<junction x="25.4" y="33.02"/>
+<pinref part="GND4" gate="1" pin="GND"/>
 </segment>
 </net>
@@
 <wire x1="63.5" y1="53.34" x2="63.5" y2="60.96" width="0.1524" layer="91"/>
 <junction x="63.5" y="53.34"/>
-<pinref part="C6" gate="G$1" pin="2"/>
+<pinref part="C3" gate="G$1" pin="+"/>
 <wire x1="63.5" y1="60.96" x2="63.5" y2="63.5" width="0.1524" layer="91"/>
 <junction x="63.5" y="60.96"/>
@@
 <wire x1="60.96" y1="88.9" x2="68.58" y2="88.9" width="0.1524" layer="91"/>
 <junction x="68.58" y="88.9"/>
-<pinref part="VAABT2" gate="VCC" pin="VCC"/>
+<pinref part="VBAT" gate="VCC" pin="VCC"/>
 <wire x1="68.58" y1="114.3" x2="71.12" y2="114.3" width="0.1524" layer="91"/>
 <wire x1="71.12" y1="114.3" x2="71.12" y2="127" width="0.1524" layer="91"/>
@@
 <wire x1="71.12" y1="134.62" x2="71.12" y2="139.7" width="0.1524" layer="91"/>
 <junction x="71.12" y="134.62"/>
-<pinref part="C3" gate="G$1" pin="+"/>
+<pinref part="C6" gate="G$1" pin="1"/>
 <junction x="71.12" y="127"/>
 </segment>
@@
 </segment>
 </net>
-<net name="N$5" class="0">
-<segment>
-<pinref part="U$3" gate="G$1" pin="PGND1@3"/>
-<wire x1="27.94" y1="35.56" x2="25.4" y2="35.56" width="0.1524" layer="91"/>
-<wire x1="25.4" y1="35.56" x2="25.4" y2="33.02" width="0.1524" layer="91"/>
-<pinref part="U$3" gate="G$1" pin="PGND2@10"/>
-<wire x1="25.4" y1="33.02" x2="25.4" y2="20.32" width="0.1524" layer="91"/>
-<wire x1="25.4" y1="20.32" x2="25.4" y2="17.78" width="0.1524" layer="91"/>
-<wire x1="25.4" y1="17.78" x2="25.4" y2="7.62" width="0.1524" layer="91"/>
-<wire x1="27.94" y1="17.78" x2="25.4" y2="17.78" width="0.1524" layer="91"/>
-<junction x="25.4" y="17.78"/>
-<pinref part="U$3" gate="G$1" pin="PGND2@9"/>
-<wire x1="27.94" y1="20.32" x2="25.4" y2="20.32" width="0.1524" layer="91"/>
-<junction x="25.4" y="20.32"/>
-<pinref part="U$3" gate="G$1" pin="PGND1@4"/>
-<wire x1="27.94" y1="33.02" x2="25.4" y2="33.02" width="0.1524" layer="91"/>
-<junction x="25.4" y="33.02"/>
-<pinref part="GND4" gate="1" pin="GND"/>
-</segment>
-<segment>
-<pinref part="U$6" gate="G$1" pin="PGND1@3"/>
-<wire x1="27.94" y1="109.22" x2="25.4" y2="109.22" width="0.1524" layer="91"/>
-<wire x1="25.4" y1="109.22" x2="25.4" y2="106.68" width="0.1524" layer="91"/>
-<pinref part="U$6" gate="G$1" pin="PGND2@10"/>
-<wire x1="25.4" y1="106.68" x2="25.4" y2="93.98" width="0.1524" layer="91"/>
-<wire x1="25.4" y1="93.98" x2="25.4" y2="91.44" width="0.1524" layer="91"/>
-<wire x1="25.4" y1="91.44" x2="25.4" y2="81.28" width="0.1524" layer="91"/>
-<wire x1="27.94" y1="91.44" x2="25.4" y2="91.44" width="0.1524" layer="91"/>
-<junction x="25.4" y="91.44"/>
-<pinref part="U$6" gate="G$1" pin="PGND2@9"/>
-<wire x1="27.94" y1="93.98" x2="25.4" y2="93.98" width="0.1524" layer="91"/>
-<junction x="25.4" y="93.98"/>
-<pinref part="U$6" gate="G$1" pin="PGND1@4"/>
-<wire x1="27.94" y1="106.68" x2="25.4" y2="106.68" width="0.1524" layer="91"/>
-<junction x="25.4" y="106.68"/>
-<pinref part="GND8" gate="1" pin="GND"/>
-</segment>
-</net>

Commit message: PsoC and MPU board finished
Other:
- moved on the sheet: LED1, R1
Changed lines of the file:
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@@
 <instance part="JP2" gate="A" x="167.64" y="76.2" rot="R180"/>
 <instance part="JP3" gate="A" x="167.64" y="35.56" rot="R180"/>
-<instance part="LED1" gate="G$1" x="248.92" y="119.38"/>
-<instance part="R1" gate="G$1" x="248.92" y="129.54" rot="R90"/>
-<instance part="SUPPLY5" gate="G$1" x="248.92" y="139.7"/>
-<instance part="GND12" gate="1" x="248.92" y="109.22"/>
+<instance part="LED1" gate="G$1" x="220.98" y="114.3"/>
+<instance part="R1" gate="G$1" x="220.98" y="124.46" rot="R90"/>
+<instance part="SUPPLY5" gate="G$1" x="220.98" y="134.62"/>
+<instance part="GND12" gate="1" x="220.98" y="104.14"/>
 <instance part="C10" gate="G$1" x="30.48" y="58.42" rot="R180"/>
 <instance part="C12" gate="G$1" x="33.02" y="129.54" rot="R180"/>
@@
 <pinref part="LED1" gate="G$1" pin="C"/>
 <pinref part="GND12" gate="1" pin="GND"/>
-<wire x1="248.92" y1="114.3" x2="248.92" y2="111.76" width="0.1524" layer="91"/>
+<wire x1="220.98" y1="109.22" x2="220.98" y2="106.68" width="0.1524" layer="91"/>
 </segment>
 <segment>
@@
 <pinref part="SUPPLY5" gate="G$1" pin="VCC"/>
 <pinref part="R1" gate="G$1" pin="2"/>
-<wire x1="248.92" y1="137.16" x2="248.92" y2="134.62" width="0.1524" layer="91"/>
+<wire x1="220.98" y1="132.08" x2="220.98" y2="129.54" width="0.1524" layer="91"/>
 </segment>
 <segment>
@@
 <pinref part="R1" gate="G$1" pin="1"/>
 <pinref part="LED1" gate="G$1" pin="A"/>
-<wire x1="248.92" y1="124.46" x2="248.92" y2="121.92" width="0.1524" layer="91"/>
-</segment>
-</net>
+<wire x1="220.98" y1="119.38" x2="220.98" y2="116.84" width="0.1524" layer="91"/>
+</segment>
+</net>

Commit message: satland production version of boards
Parts:
- added R2: (no value), rcl:R-EU_R0805
- added X2: (no value), con-ptr500:AK500/2
Connections:
- new net BAT: JP1.3, JP1.4, R2.1, U$4.1_IN+, U$4.2_IN+, X1-1.KL
- net GND: now also X2-2.KL
- net VCC: now also R2.2, X2-1.KL; no longer JP1.3, JP1.4, U$4.1_IN+, U$4.2_IN+, X1-1.KL
Changed lines of the file:
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@@
 <part name="C7" library="rcl" deviceset="CPOL-EU" device="153CLV-0405" value="10u"/>
 <part name="GND3" library="supply1" deviceset="GND" device=""/>
-<part name="VAABT3" library="supply1" deviceset="VCC" device="" value="VBAT"/>
 <part name="C3" library="rcl" deviceset="CPOL-EU" device="153CLV-0405" value="10u"/>
 <part name="C6" library="rcl" deviceset="C-EU" device="C0603" value="100n"/>
 <part name="GND8" library="supply1" deviceset="GND" device=""/>
 <part name="GND4" library="supply1" deviceset="GND" device=""/>
+<part name="X2" library="con-ptr500" deviceset="AK500/2" device=""/>
+<part name="GND15" library="supply1" deviceset="GND" device=""/>
+<part name="R2" library="rcl" deviceset="R-EU_" device="R0805"/>
+<part name="VAABT2" library="supply1" deviceset="VCC" device="" value="VBAT"/>
 </parts>
 <sheets>
@@
 <instance part="GND2" gate="1" x="195.58" y="109.22"/>
 <instance part="SUPPLY1" gate="G$1" x="195.58" y="134.62"/>
-<instance part="VAABT" gate="VCC" x="132.08" y="137.16"/>
+<instance part="VAABT" gate="VCC" x="132.08" y="165.1"/>
 <instance part="GND5" gate="1" x="63.5" y="5.08"/>
 <instance part="SUPPLY3" gate="G$1" x="63.5" y="66.04"/>
@@
 <instance part="C7" gate="G$1" x="60.96" y="134.62" rot="R270"/>
 <instance part="GND3" gate="1" x="127" y="10.16"/>
-<instance part="VAABT3" gate="VCC" x="152.4" y="27.94"/>
 <instance part="C3" gate="G$1" x="60.96" y="60.96" rot="R270"/>
 <instance part="C6" gate="G$1" x="73.66" y="127" rot="R90"/>
 <instance part="GND8" gate="1" x="25.4" y="78.74"/>
 <instance part="GND4" gate="1" x="25.4" y="5.08"/>
+<instance part="X2" gate="-1" x="124.46" y="160.02"/>
+<instance part="X2" gate="-2" x="124.46" y="154.94"/>
+<instance part="GND15" gate="1" x="132.08" y="149.86"/>
+<instance part="R2" gate="G$1" x="147.32" y="137.16"/>
+<instance part="VAABT2" gate="VCC" x="154.94" y="142.24"/>
 </instances>
 <busses>
@@
 <pinref part="GND4" gate="1" pin="GND"/>
 </segment>
+<segment>
+<pinref part="X2" gate="-2" pin="KL"/>
+<pinref part="GND15" gate="1" pin="GND"/>
+<wire x1="129.54" y1="154.94" x2="132.08" y2="154.94" width="0.1524" layer="91"/>
+<wire x1="132.08" y1="154.94" x2="132.08" y2="152.4" width="0.1524" layer="91"/>
+</segment>
 </net>
 <net name="VCC" class="0">
-<segment>
-<pinref part="U$4" gate="G$1" pin="1_IN+"/>
-<pinref part="X1" gate="-1" pin="KL"/>
-<wire x1="137.16" y1="129.54" x2="132.08" y2="129.54" width="0.1524" layer="91"/>
-<pinref part="U$4" gate="G$1" pin="2_IN+"/>
-<wire x1="137.16" y1="127" x2="132.08" y2="127" width="0.1524" layer="91"/>
-<wire x1="132.08" y1="127" x2="132.08" y2="129.54" width="0.1524" layer="91"/>
-<junction x="132.08" y="129.54"/>
-<pinref part="VAABT" gate="VCC" pin="VCC"/>
-<wire x1="132.08" y1="129.54" x2="132.08" y2="134.62" width="0.1524" layer="91"/>
-<wire x1="132.08" y1="129.54" x2="124.46" y2="129.54" width="0.1524" layer="91"/>
-</segment>
 <segment>
 <pinref part="U$4" gate="G$1" pin="1_OUT+"/>
@@
 </segment>
 <segment>
-<pinref part="JP1" gate="A" pin="3"/>
-<wire x1="114.3" y1="22.86" x2="124.46" y2="22.86" width="0.1524" layer="91"/>
-<wire x1="124.46" y1="22.86" x2="152.4" y2="22.86" width="0.1524" layer="91"/>
-<wire x1="152.4" y1="22.86" x2="152.4" y2="25.4" width="0.1524" layer="91"/>
-<pinref part="JP1" gate="A" pin="4"/>
-<wire x1="114.3" y1="25.4" x2="124.46" y2="25.4" width="0.1524" layer="91"/>
-<wire x1="124.46" y1="25.4" x2="124.46" y2="22.86" width="0.1524" layer="91"/>
-<junction x="124.46" y="22.86"/>
-<pinref part="VAABT3" gate="VCC" pin="VCC"/>
+<pinref part="X2" gate="-1" pin="KL"/>
+<pinref part="VAABT" gate="VCC" pin="VCC"/>
+<wire x1="129.54" y1="160.02" x2="132.08" y2="160.02" width="0.1524" layer="91"/>
+<wire x1="132.08" y1="160.02" x2="132.08" y2="162.56" width="0.1524" layer="91"/>
+</segment>
+<segment>
+<pinref part="R2" gate="G$1" pin="2"/>
+<wire x1="152.4" y1="137.16" x2="154.94" y2="137.16" width="0.1524" layer="91"/>
+<wire x1="154.94" y1="137.16" x2="154.94" y2="139.7" width="0.1524" layer="91"/>
+<pinref part="VAABT2" gate="VCC" pin="VCC"/>
 </segment>
 </net>
@@
 </segment>
 </net>
+<net name="BAT" class="0">
+<segment>
+<pinref part="U$4" gate="G$1" pin="1_IN+"/>
+<pinref part="X1" gate="-1" pin="KL"/>
+<wire x1="137.16" y1="129.54" x2="132.08" y2="129.54" width="0.1524" layer="91"/>
+<pinref part="U$4" gate="G$1" pin="2_IN+"/>
+<wire x1="137.16" y1="127" x2="132.08" y2="127" width="0.1524" layer="91"/>
+<wire x1="132.08" y1="127" x2="132.08" y2="129.54" width="0.1524" layer="91"/>
+<junction x="132.08" y="129.54"/>
+<wire x1="132.08" y1="129.54" x2="124.46" y2="129.54" width="0.1524" layer="91"/>
+<wire x1="132.08" y1="129.54" x2="132.08" y2="137.16" width="0.1524" layer="91"/>
+<wire x1="132.08" y1="137.16" x2="142.24" y2="137.16" width="0.1524" layer="91"/>
+<pinref part="R2" gate="G$1" pin="1"/>
+<wire x1="132.08" y1="137.16" x2="127" y2="137.16" width="0.1524" layer="91"/>
+<junction x="132.08" y="137.16"/>
+<label x="127" y="137.16" size="1.778" layer="95" rot="R180" xref="yes"/>
+</segment>
+<segment>
+<pinref part="JP1" gate="A" pin="3"/>
+<wire x1="114.3" y1="22.86" x2="124.46" y2="22.86" width="0.1524" layer="91"/>
+<wire x1="124.46" y1="22.86" x2="134.62" y2="22.86" width="0.1524" layer="91"/>
+<pinref part="JP1" gate="A" pin="4"/>
+<wire x1="114.3" y1="25.4" x2="124.46" y2="25.4" width="0.1524" layer="91"/>
+<wire x1="124.46" y1="25.4" x2="124.46" y2="22.86" width="0.1524" layer="91"/>
+<junction x="124.46" y="22.86"/>
+<label x="134.62" y="22.86" size="1.778" layer="95" xref="yes"/>
+</segment>
+</net>
